Commit message: Update: namespace distinguishion

File: dsr_description2/config/macro.gazebo.xacro (robot description, xacro)
@@ -6,5 +6,9 @@
     <gazebo>
       <plugin filename="ign_ros2_control-system" name="ign_ros2_control::IgnitionROS2ControlPlugin">
+        <ros>
+          <namespace>$(arg namespace)</namespace>
+        </ros>
         <parameters>$(find dsr_controller2)/config/dsr_controller2_gz.yaml</parameters>
+        <!-- <controller_manager_name>asd</controller_manager_name> -->
       </plugin>
     </gazebo>

File: dsr_description2/ros2_control/m1013.gz_ros2_control.xacro (robot description, xacro)
@@ -25,5 +25,5 @@
           <plugin>ign_ros2_control/IgnitionSystem</plugin>
       </hardware>
-      <joint name="${namespace}joint_1">
+      <joint name="joint_1">
         <command_interface name="position">
           <param name="min">{-2*pi}</param>
@@ -35,5 +35,5 @@
         <state_interface name="velocity"/>
       </joint>
-      <joint name="${namespace}joint_2">
+      <joint name="joint_2">
         <command_interface name="position">
           <param name="min">{-2*pi}</param>
@@ -45,5 +45,5 @@
         <state_interface name="velocity"/>
       </joint>
-      <joint name="${namespace}joint_3">
+      <joint name="joint_3">
         <command_interface name="position">
           <param name="min">{-pi}</param>
@@ -55,5 +55,5 @@
         <state_interface name="velocity"/>
       </joint>
-      <joint name="${namespace}joint_4">
+      <joint name="joint_4">
         <command_interface name="position">
           <param name="min">{-2*pi}</param>
@@ -65,5 +65,5 @@
         <state_interface name="velocity"/>
       </joint>
-      <joint name="${namespace}joint_5">
+      <joint name="joint_5">
         <command_interface name="position">
           <param name="min">{-2*pi}</param>
@@ -75,5 +75,5 @@
         <state_interface name="velocity"/>
       </joint>
-      <joint name="${namespace}joint_6">
+      <joint name="joint_6">
         <command_interface name="position">
           <param name="min">{-2*pi}</param>
