Commit message: fix: xacro collision error

File: dsr_description2/ros2_control/m0609.gz_ros2_control.xacro (robot description, xacro)
@@ -15,10 +15,4 @@
   use_gazebo:=false
   ">
-    <xacro:include filename="$(find dsr_description2)/config/macro.gazebo.xacro" />
-    <xacro:include filename="$(find dsr_description2)/config/macro.transmission.xacro" />
-    <xacro:include filename="$(find dsr_description2)/config/macro.materials.xacro" />
-    <xacro:dsr_materials />
-    <xacro:dsr_transmission />
-    <xacro:dsr_gazebo namespace="${namespace}" />
     <ros2_control name="${model}" type="system">
       <hardware>

File: dsr_description2/ros2_control/m0617.gz_ros2_control.xacro (robot description, xacro)
@@ -15,10 +15,4 @@
   use_gazebo:=false
   ">
-    <xacro:include filename="$(find dsr_description2)/config/macro.gazebo.xacro" />
-    <xacro:include filename="$(find dsr_description2)/config/macro.transmission.xacro" />
-    <xacro:include filename="$(find dsr_description2)/config/macro.materials.xacro" />
-    <xacro:dsr_materials />
-    <xacro:dsr_transmission />
-    <xacro:dsr_gazebo namespace="${namespace}" />
     <ros2_control name="${model}" type="system">
       <hardware>

File: dsr_description2/ros2_control/m1013.gz_ros2_control.xacro (robot description, xacro)
@@ -15,10 +15,4 @@
   use_gazebo:=false
   ">
-    <xacro:include filename="$(find dsr_description2)/config/macro.gazebo.xacro" />
-    <xacro:include filename="$(find dsr_description2)/config/macro.transmission.xacro" />
-    <xacro:include filename="$(find dsr_description2)/config/macro.materials.xacro" />
-    <xacro:dsr_materials />
-    <xacro:dsr_transmission />
-    <xacro:dsr_gazebo namespace="${namespace}" />
     <ros2_control name="${model}" type="system">
       <hardware>

File: dsr_description2/ros2_control/m1509.gz_ros2_control.xacro (robot description, xacro)
@@ -15,10 +15,4 @@
   use_gazebo:=false
   ">
-    <xacro:include filename="$(find dsr_description2)/config/macro.gazebo.xacro" />
-    <xacro:include filename="$(find dsr_description2)/config/macro.transmission.xacro" />
-    <xacro:include filename="$(find dsr_description2)/config/macro.materials.xacro" />
-    <xacro:dsr_materials />
-    <xacro:dsr_transmission />
-    <xacro:dsr_gazebo namespace="${namespace}" />
     <ros2_control name="${model}" type="system">
       <hardware>

File: dsr_description2/xacro/macro.e0509.white.xacro (robot description, xacro)
@@ -17,4 +17,5 @@
 					<mesh filename="package://dsr_description2/meshes/e0509_collision/E0509_0_0.dae" scale="0.001 0.001 0.001" />
 				</geometry>
+				<material name="dr_white" />
 			</collision>
 			<visual>
@@ -23,4 +24,5 @@
 					<mesh filename="package://dsr_description2/meshes/e0509_white/E0509_0_0.dae" scale="0.001 0.001 0.001" />
 				</geometry>
+				<material name="dr_white" />
 			</visual>
 		</link>
@@ -32,60 +34,69 @@
       <axis xyz="0 0 1"/>
       <limit effort="194" lower="-6.2832" upper="6.2832" velocity="3.1416"/>
-			<dynamics friction="0" />
+		<dynamics friction="0" />
 		</joint>
 		<link name="link_1">
-			<inertial>
-        <mass value="5.75"/>
-        <origin xyz="1e-06    0.049633   -0.049635"/>
-        <inertia ixx="0.046214" ixy="1.4982e-05" ixz="1.281e-05" iyy="0.032573" iyz="-0.013997" izz="0.030999"/>
-      </inertial>
-            <collision>
-				<origin rpy="0 0 0" xyz="0 0 0" />
-				<geometry>
-					<mesh filename="package://dsr_description2/meshes/e0509_collision/E0509_1_1.dae" scale="0.001 0.001 0.001" />
-				</geometry>
-			</collision>
+		<inertial>
+			<mass value="5.75"/>
+			<origin xyz="1e-06    0.049633   -0.049635"/>
+			<inertia ixx="0.046214" ixy="1.4982e-05" ixz="1.281e-05" iyy="0.032573" iyz="-0.013997" izz="0.030999"/>
+		</inertial>
+		<collision>
+			<origin rpy="0 0 0" xyz="0 0 0" />
+			<geometry>
+				<mesh filename="package://dsr_description2/meshes/e0509_collision/E0509_1_1.dae" scale="0.001 0.001 0.001"
+				/>
+			</geometry>
+			<material name="dr_white" />
+		</collision>
       		<visual>
-				<origin rpy="0 0 0" xyz="0 0 0" />
-				<geometry>
-					<mesh filename="package://dsr_description2/meshes/e0509_white/E0509_1_1.dae" scale="0.001 0.001 0.001" />
-				</geometry>
-			</visual>
-			<collision>
-				<origin rpy="0 0 0" xyz="0 0 0" />
-				<geometry>
-					<mesh filename="package://dsr_description2/meshes/e0509_collision/E0509_1_2.dae" scale="0.001 0.001 0.001" />
-				</geometry>
-			</collision>
-            <visual>
-				<origin rpy="0 0 0" xyz="0 0 0" />
-				<geometry>
-					<mesh filename="package://dsr_description2/meshes/e0509_white/E0509_1_2.dae" scale="0.001 0.001 0.001" />
-				</geometry>
-			</visual>
-			<collision>
-				<origin rpy="0 0 0" xyz="0 0 0" />
-				<geometry>
-					<mesh filename="package://dsr_description2/meshes/e0509_collision/E0509_1_3.dae" scale="0.001 0.001 0.001" />
-				</geometry>
-			</collision>
+			<origin rpy="0 0 0" xyz="0 0 0" />
+			<geometry>
+				<mesh filename="package://dsr_description2/meshes/e0509_white/E0509_1_1.dae" scale="0.001 0.001 0.001" />
+			</geometry>
+			<material name="dr_white" />
+		</visual>
+		<collision>
+			<origin rpy="0 0 0" xyz="0 0 0" />
+			<geometry>
+				<mesh filename="package://dsr_description2/meshes/e0509_collision/E0509_1_2.dae" scale="0.001 0.001 0.001" />
+			</geometry>
+			<material name="dr_white" />
+		</collision>
+		<visual>
+			<origin rpy="0 0 0" xyz="0 0 0" />
+			<geometry>
+				<mesh filename="package://dsr_description2/meshes/e0509_white/E0509_1_2.dae" scale="0.001 0.001 0.001" />
+			</geometry>
+			<material name="dr_white" />
+		</visual>
+		<collision>
+			<origin rpy="0 0 0" xyz="0 0 0" />
+			<geometry>
+				<mesh filename="package://dsr_description2/meshes/e0509_collision/E0509_1_3.dae" scale="0.001 0.001 0.001" />
+			</geometry>
+			<material name="dr_white" />
+		</collision>
       		<visual>
-				<origin rpy="0 0 0" xyz="0 0 0" />
-				<geometry>
-					<mesh filename="package://dsr_description2/meshes/e0509_white/E0509_1_3.dae" scale="0.001 0.001 0.001" />
-				</geometry>
-			</visual>
-			<collision>
-				<origin rpy="0 0 0" xyz="0 0 0" />
-				<geometry>
-					<mesh filename="package://dsr_description2/meshes/e0509_collision/E0509_1_4.dae" scale="0.001 0.001 0.001" />
-				</geometry>
-			</collision>
-            <visual>
-				<origin rpy="0 0 0" xyz="0 0 0" />
-				<geometry>
-					<mesh filename="package://dsr_description2/meshes/e0509_white/E0509_1_4.dae" scale="0.001 0.001 0.001" />
-				</geometry>
-			</visual>
+			<origin rpy="0 0 0" xyz="0 0 0" />
+			<geometry>
+				<mesh filename="package://dsr_description2/meshes/e0509_white/E0509_1_3.dae" scale="0.001 0.001 0.001" />
+			</geometry>
+			<material name="dr_white" />
+		</visual>
+		<collision>
+			<origin rpy="0 0 0" xyz="0 0 0" />
+			<geometry>
+				<mesh filename="package://dsr_description2/meshes/e0509_collision/E0509_1_4.dae" scale="0.001 0.001 0.001" />
+			</geometry>
+			<material name="dr_white" />
+		</collision>
+            	<visual>
+			<origin rpy="0 0 0" xyz="0 0 0" />
+			<geometry>
+				<mesh filename="package://dsr_description2/meshes/e0509_white/E0509_1_4.dae" scale="0.001 0.001 0.001" />
+			</geometry>
+			<material name="dr_white" />
+		</visual>
 		</link>
 		<!-- joint2 -->
@@ -109,4 +120,5 @@
 					<mesh filename="package://dsr_description2/meshes/e0509_collision/E0509_2_1.dae" scale="0.001 0.001 0.001" />
 				</geometry>
+				<material name="dr_white" />
 			</collision>
 			<visual>
@@ -115,4 +127,5 @@
 					<mesh filename="package://dsr_description2/meshes/e0509_white/E0509_2_1.dae" scale="0.001 0.001 0.001" />
 				</geometry>
+				<material name="dr_white" />
 			</visual>
 			<collision>
@@ -121,4 +134,5 @@
 					<mesh filename="package://dsr_description2/meshes/e0509_collision/E0509_2_2.dae" scale="0.001 0.001 0.001" />
 				</geometry>
+				<material name="dr_white" />
 			</collision>
 			<visual>
@@ -127,4 +141,5 @@
 					<mesh filename="package://dsr_description2/meshes/e0509_white/E0509_2_2.dae" scale="0.001 0.001 0.001" />
 				</geometry>
+				<material name="dr_white" />
 			</visual>
 		</link>
@@ -149,4 +164,5 @@
 					<mesh filename="package://dsr_description2/meshes/e0509_collision/E0509_3_1.dae" scale="0.001 0.001 0.001" />
 				</geometry>
+				<material name="dr_white" />
 			</collision>
 			<visual>
@@ -155,4 +171,5 @@
 					<mesh filename="package://dsr_description2/meshes/e0509_white/E0509_3_1.dae" scale="0.001 0.001 0.001" />
 				</geometry>
+				<material name="dr_white" />
 			</visual>
 			<collision>
@@ -161,4 +178,5 @@
 					<mesh filename="package://dsr_description2/meshes/e0509_collision/E0509_3_2.dae" scale="0.001 0.001 0.001" />
 				</geometry>
+				<material name="dr_white" />
 			</collision>
             <visual>
@@ -167,4 +185,5 @@
 					<mesh filename="package://dsr_description2/meshes/e0509_white/E0509_3_2.dae" scale="0.001 0.001 0.001" />
 				</geometry>
+				<material name="dr_white" />
 			</visual>
 		</link>
@@ -189,4 +208,5 @@
 					<mesh filename="package://dsr_description2/meshes/e0509_collision/E0509_4_1.dae" scale="0.001 0.001 0.001" />
 				</geometry>
+				<material name="dr_white" />
 			</collision>
 			<visual>
@@ -195,4 +215,5 @@
 					<mesh filename="package://dsr_description2/meshes/e0509_white/E0509_4_1.dae" scale="0.001 0.001 0.001" />
 				</geometry>
+				<material name="dr_white" />
 			</visual>
 			<collision>
@@ -201,4 +222,5 @@
 					<mesh filename="package://dsr_description2/meshes/e0509_collision/E0509_4_2.dae" scale="0.001 0.001 0.001" />
 				</geometry>
+				<material name="dr_white" />
 			</collision>
 			<visual>
@@ -207,4 +229,5 @@
 					<mesh filename="package://dsr_description2/meshes/e0509_white/E0509_4_2.dae" scale="0.001 0.001 0.001" />
 				</geometry>
+				<material name="dr_white" />
 			</visual>
 		</link>
@@ -229,4 +252,5 @@
 					<mesh filename="package://dsr_description2/meshes/e0509_collision/E0509_5_1.dae" scale="0.001 0.001 0.001" />
 				</geometry>
+				<material name="dr_white" />
 			</collision>
 			<visual>
@@ -235,4 +259,5 @@
 					<mesh filename="package://dsr_description2/meshes/e0509_white/E0509_5_1.dae" scale="0.001 0.001 0.001" />
 				</geometry>
+				<material name="dr_white" />
 			</visual>
 			<collision>
@@ -241,4 +266,5 @@
 					<mesh filename="package://dsr_description2/meshes/e0509_collision/E0509_5_2.dae" scale="0.001 0.001 0.001" />
 				</geometry>
+				<material name="dr_white" />
 			</collision>
             <visual>
@@ -247,4 +273,5 @@
 					<mesh filename="package://dsr_description2/meshes/e0509_white/E0509_5_2.dae" scale="0.001 0.001 0.001" />
 				</geometry>
+				<material name="dr_white" />
 			</visual>
 		</link>
@@ -269,4 +296,5 @@
 					<mesh filename="package://dsr_description2/meshes/e0509_collision/E0509_6_1.dae" scale="0.001 0.001 0.001" />
 				</geometry>
+				<material name="dr_white" />
 			</collision>
 			<visual>
@@ -275,4 +303,5 @@
 					<mesh filename="package://dsr_description2/meshes/e0509_white/E0509_6_1.dae" scale="0.001 0.001 0.001" />
 				</geometry>
+				<material name="dr_white" />
 			</visual>
 		</link>
